File: Hardware/Kicad3/Faderbay/Faderbay.kicad_sch (KiCad schematic)
At the start: 201 parts, among them U1 STM32F405RGTx

Commit message: Schematic updates
Connections:
- net +3.3V: now also C?.1, C?.1, C?.1, C?.1, U?.11 (V-), U?.11 (V-), U?.11 (V-), U?.11 (V-); no longer C?.2, C?.2, C?.2, C?.2, U?.4 (V+), U?.4 (V+), U?.4 (V+), U?.4 (V+)
- net GND: now also C?.2, C?.2, C?.2, C?.2, U?.4 (V+), U?.4 (V+), U?.4 (V+), U?.4 (V+); no longer C?.1, C?.1, C?.1, C?.1, U?.11 (V-), U?.11 (V-), U?.11 (V-), U?.11 (V-)
- net UART3_TX: no longer U1.29 (PB10)
- net UART1_RX: no longer names the net of U1.43 (PA10)
- net UART1_TX: no longer names the net of U1.42 (PA9)
- net UART3_RX: no longer names the net of U1.30 (PB11)
- new net UART_TX: U1.29 (PB10)
- no-connect marks 62 -> 65
Other:
- moved on the sheet: C?, J?
