File: Hardware/Kicad/Faderbay_12V.kicad_sch (KiCad schematic)
At the start: 176 parts, among them J14 MIDI DIN-5, J2 USB_C_Receptacle_USB2.0_14P, J3 SWD, J4 52437-2471, Q2 MMBT2222A, SW1 SW_Push_Dual, SW2 SW_Push_Dual, SW3 EC11E15204A3, SW4 SW_Push_Dual, SW5 SW_Push_Dual, U1 USBLC6-2SC6, U10 TL074, U4 STM32F405RGTx, U5 CD74HC4067M, U6 TL074, U7 TL074, U8 MCP6002, U9 TL074, Y1 16MHz

Commit message: Commit
Parts:
- removed C? (x2): 100u, symbol Device:C_Small
- removed C? (x5): 10u, symbol Device:C_Small
- removed C? (x4): 100n, symbol Device:C_Small
- removed F?: 750mA, symbol Device:Fuse_Small
- removed J?: UART, symbol Connector:Conn_01x02_Pin
- removed R? (x2): 0, symbol Device:R_Small
- removed TP? (x11): TestPoint, symbol Connector:TestPoint
- removed U?: ICL7660, symbol Regulator_SwitchedCapacitor:ICL7660
- removed U?: TLV75733PDBV, Package_TO_SOT_SMD:SOT-23-5, symbol Regulator_Linear:TLV75733PDBV
- added C10, C11: 2.2u, Capacitor_SMD:C_1206_3216Metric, symbol Device:C_Small
- added C13, C14: 100n, Capacitor_SMD:C_0402_1005Metric, symbol Device:C_Small
- added C15, C16, C17, C18: 22u, Capacitor_SMD:C_1206_3216Metric, symbol Device:C_Small
- added J1: Barrel_Jack_Switch, Connector_BarrelJack:BarrelJack_Kycon_KLDX-0202-xC_Horizontal, symbol Connector:Barrel_Jack_Switch
- added L1: 6.8u, Inductor_SMD:L_Changjiang_FXL0530, symbol Device:L_Small
- added L2: 5.6u, Inductor_SMD:L_Changjiang_FXL0630, symbol Device:L_Small
- added Q1: AO3401A, Package_TO_SOT_SMD:SOT-23, symbol Transistor_FET:AO3401A
- added R10: 22.1k, Resistor_SMD:R_0603_1608Metric, symbol Device:R_Small
- added R7, R9: 100k, Resistor_SMD:R_0603_1608Metric, symbol Device:R_Small
- added R8: 13.7k, Resistor_SMD:R_0603_1608Metric, symbol Device:R_Small
- added U2, U3: LMR51430, Package_TO_SOT_SMD:SOT-23-6, symbol Regulator_Switching:LMR51430
- FB1: value 100@100MHz -> 600 @ 6600MHz; Assembly (none) -> Y; LCSC Part # (none) -> C1017
Connections:
- net +5VA is gone; now on net +12V: FB1.2
- net GNDD is gone; now on net GND: C1.2, C12.2, C2.2, C20.2, C21.2, C22.2, C27.2, C29.2, C3.2, C4.2, C5.2, C6.2, C7.2, C8.2, C9.2, D2.1 (K), D3.1 (K), J14.2, J3.3 (Pin_3), J3.5 (Pin_5), J3.9 (Pin_9), J4.1, J4.11, J4.12, J4.16, J4.17, J4.18, J4.19, J4.2, J4.20, J4.24, J4.3, J4.6, J4.7, J9.1, Q2.2 (E), R60.1, R61.1, R67.1, R68.1, R69.1, SW3.C1, SW3.MH1, SW3.MH2, U1.2 (GND), U4.12 (VSSA), U4.18 (VSS), U4.60 (BOOT0), U4.63 (VSS), U5.12 (GND), U8.4 (V-), U8.9 (V-), Y1.2, Y1.4
- net +12V: now also C10.2, C11.2, U2.3 (VIN), U2.5 (EN), U3.3 (VIN), U3.5 (EN)
- net +3.3V: now also C16.2, C18.2, L2.2, R9.2
- net +5V: now also C15.2, C17.2, L1.2, R7.2
- net GND: now also S1.5 (COM_2), S1.MH1, S1.MH2, C10.1, C11.1, C15.1, C16.1, C17.1, C18.1, Q1.1 (G), R10.1, R8.1, U2.1 (GND), U3.1 (GND)
- net USB_VBUS: now also J2.A4 (VBUS), J2.A9 (VBUS), J2.B4 (VBUS), J2.B9 (VBUS)
- net 12V_In: now reaches S1.2 (COM_1)
- net 12V_In: now also Q1.3 (D)
- net at S1.6 (NO_2): now also J1.2, J1.3
- net +5VD: no longer names the net of S1.1 (NO_1)
- net +5VD: now also J1.1; no longer FB1.1
- new net: C14.1, L2.1, U3.2 (SW)
- new net: R10.2, R9.1, U3.4 (FB)
- new net: C14.2, U3.6 (CB)
- new net: R7.1, R8.2, U2.4 (FB)
- new net: C13.1, L1.1, U2.2 (SW)
- new net: C13.2, U2.6 (CB)
- new net: FB1.1, Q1.2 (S)
- no-connect marks 46 -> 40
Other:
- moved on the sheet: C19, FB1, H1, H2, H3, H4, J2, R2, R3, RV1, RV10, RV11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
