File: Hardware/Kicad/Faderbay.kicad_sch (KiCad schematic)
At the start: 176 parts, among them J14 MIDI DIN-5, J2 USB_C_Receptacle_USB2.0_14P, J3 SWD, J4 52437-2471, Q2 MMBT2222A, SW1 SW_Push_Dual, SW2 SW_Push_Dual, SW3 EC11E15204A3, SW4 SW_Push_Dual, SW5 SW_Push_Dual, U1 USBLC6-2SC6, U10 TL074, U4 STM32F405RGTx, U5 CD74HC4067M, U6 TL074, U7 TL074, U8 MCP6002, U9 TL074, Y1 16MHz

Commit message: 18/01/26
Parts:
- removed C20, C23, C24, C25, C26: 100n, Capacitor_SMD:C_0402_1005Metric, symbol Device:C_Small
- removed C21: 1u, Capacitor_SMD:C_0402_1005Metric, symbol Device:C_Small
- removed C22: 10n, Capacitor_SMD:C_0402_1005Metric, symbol Device:C_Small
- removed J10, J11, J12, J13, J15, J16, J17, J18, J19, J20, J21, J22, J6, J7, J8: ~, Eurorack:BOOMELE_PJ-320B, symbol Eurorack:PJ-320B
- removed L3: 39n, Inductor_SMD:L_0402_1005Metric, symbol Device:L_Small
- removed R11, R12, R13, R14, R15, R16, R29, R30, R31, R32, R33, R34, R47, R48, R49, R50: 10k, Resistor_SMD:R_0603_1608Metric, symbol Device:R_Small
- removed R17, R18, R19, R20, R21, R22, R35, R36, R37, R38, R39, R40, R51, R52, R53, R54: 20k, Resistor_SMD:R_0603_1608Metric, symbol Device:R_Small
- removed R23, R24, R25, R26, R27, R28, R41, R42, R43, R44, R45, R46, R55, R56, R57, R58: 1k, Resistor_SMD:R_0603_1608Metric, symbol Device:R_Small
- removed R65: 10k, Resistor_SMD:R_0402_1005Metric, symbol Device:R_Small
- removed RV1, RV10, RV11, RV12, RV13, RV14, RV15, RV16, RV2, RV3, RV4, RV5, RV6, RV7, RV8, RV9: R_Potentiometer, User:PTB60442010BPA104, symbol Device:R_Potentiometer
- removed TP? (x2): TestPoint, symbol Connector:TestPoint
- removed U10, U6, U7, U9: TL074, Package_SO:SOIC-14_3.9x8.7mm_P1.27mm, symbol Amplifier_Operational:TL074
- removed U8: MCP6002, Package_SO:SOIC-8_3.9x4.9mm_P1.27mm, symbol Amplifier_Operational:MCP6002-xMC
- added C? (x9): 100n, symbol Device:C_Small
- added C?: 100n, Capacitor_SMD:C_0402_1005Metric, symbol Device:C_Small
- added C?: 10n, Capacitor_SMD:C_0402_1005Metric, symbol Device:C_Small
- added C?: 10u, Capacitor_SMD:C_0402_1005Metric, symbol Device:C_Small
- added FB? (x2): 100@100MHz, Inductor_SMD:L_0805_2012Metric, symbol Device:FerriteBead_Small
- added J? (x15): ~, Eurorack:BOOMELE_PJ-320B, symbol Eurorack:PJ-320B
- added R? (x32): 10k, symbol Device:R_Small
- added R? (x16): 1k, symbol Device:R_Small
- added R? (x2): 220, Resistor_SMD:R_0603_1608Metric, symbol Device:R_Small
- added RV? (x16): 100k, User:PTB60442010BPA104, symbol Device:R_Potentiometer
- added TP? (x2): TestPoint, symbol Connector:TestPoint
- added U? (x20): MCP6004, symbol Amplifier_Operational:MCP6004
- added U?: MCP6001-OT, Package_TO_SOT_SMD:SOT-23-5, symbol Amplifier_Operational:MCP6001-OT
- R4: value 560 -> 230
- R64: value 10k -> 1k
Connections:
- net +12V: no longer R4.2
- net +3.3V: now also C?.1, FB?.1, U?.2 (V-)
- net +5V: now also R4.2, R?.1
- net +5VA: now also U?.7 (OSC), C?.1, C?.1, C?.1, C?.1, R?.1, R?.1, R?.1, R?.1, R?.1, R?.1, R?.1, R?.1, R?.1, R?.1, R?.1, R?.1, R?.1, R?.1, R?.1, R?.1, RV?.1, RV?.1, RV?.1, RV?.1, RV?.1, RV?.1, RV?.1, RV?.1, RV?.1, RV?.1, RV?.1, RV?.1, RV?.1, RV?.1, RV?.1, RV?.1, U?.4 (V+), U?.4 (V+), U?.4 (V+), U?.4 (V+)
- net -5VA: now also C?.1, C?.1, C?.1, C?.1, FB?.2, U?.11 (V-), U?.11 (V-), U?.11 (V-), U?.11 (V-); no longer U?.5 (VOUT)
- net ADC_BUFF: now also U?.3 (+)
- net ADC_IN: now also TP?.1, U?.1, U?.4 (-)
- net GND: no longer J5.1, J5.2
- net GNDA: now also J5.1, J5.2, U4.12 (VSSA), C?.2, C?.2, C?.2, C?.2, C?.2, C?.2, C?.2, C?.2, C?.2, C?.2, J?.1, J?.1, J?.1, J?.1, J?.1, J?.1, J?.1, J?.1, J?.1, J?.1, J?.1, J?.1, J?.1, J?.1, J?.1, J?.2, J?.2, J?.2, J?.2, J?.2, J?.2, J?.2, J?.2, J?.2, J?.2, J?.2, J?.2, J?.2, J?.2, J?.2, RV?.3, RV?.3, RV?.3, RV?.3, RV?.3, RV?.3, RV?.3, RV?.3, RV?.3, RV?.3, RV?.3, RV?.3, RV?.3, RV?.3, RV?.3, RV?.3
- net GNDD: now also C?.2, U?.5 (V+); no longer J14.2, U4.12 (VSSA)
- net P0: now also RV?.2, U?.3 (+)
- net P1: now also RV?.2, U?.5 (+)
- net P10: now also RV?.2, U?.10 (+)
- net P11: now also RV?.2, U?.12 (+)
- net P12: now also RV?.2, U?.3 (+)
- net P13: now also RV?.2, U?.5 (+)
- net P14: now also RV?.2, U?.10 (+)
- net P15: now also RV?.2, U?.12 (+)
- net P2: now also RV?.2, U?.10 (+)
- net P3: now also RV?.2, U?.12 (+)
- net P4: now also RV?.2, U?.3 (+)
- net P5: now also RV?.2, U?.5 (+)
- net P6: now also RV?.2, U?.10 (+)
- net P7: now also RV?.2, U?.12 (+)
- net P8: now also RV?.2, U?.3 (+)
- net P9: now also RV?.2, U?.5 (+)
- net VDDA: now also C?.1, C?.2, TP?.1
- net J0: no longer names the net of J5.3
- net J0: now also R?.2
- net MIDI_OUT: no longer names the net of Q2.3 (C), R66.1
- net MIDI_OUT: now also R?.1
- net MIDI_TRS_R: no longer names the net of J14.4, R63.1
- net MIDI_TRS_R: no longer J9.2
- net MIDI_TRS_T: no longer names the net of J14.5, R66.2
- net MIDI_TRS_T: no longer J9.3
- new net: J?.3, R?.2 (x15)
- new net: R?.1, R?.2, U?.2 (-) (x4)
- new net: R?.1, R?.2, U?.1 (x4)
- new net: R?.1, R?.2, U?.8 (x4)
- new net: R?.1, R?.2, U?.7 (x4)
- new net: R?.1, R?.2, U?.6 (-) (x4)
- new net: R?.1, R?.2, U?.13 (-) (x4)
- new net: R?.1, R?.2, U?.14 (x4)
- new net: C?.1, C?.1, FB?.2
- new net: J9.2, R?.2
- new net: R?.1, R?.2, U?.9 (-) (x4)
- new net: J9.3, R?.2
- new net: FB?.1, U?.5 (VOUT)
Other:
- note added: "MIDI TRS Type A"
- note removed: "FADERS"
- note removed: "JACK CONNECTORS"
- moved on the sheet: C?, FB1, H1, H2, H3, H4, J14, J5, J9, Q2, R59, R60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

Commit message: 31/01/26
Parts:
- removed C27: 4,7u, Capacitor_SMD:C_0402_1005Metric, symbol Device:C_Small
- removed C28, C29: 100n, Capacitor_SMD:C_0402_1005Metric, symbol Device:C_Small
- removed J4: 52437-2471, User:524372471, symbol User:52437-2471
- removed R69: 910k, Resistor_SMD:R_0402_1005Metric, symbol Device:R_Small
- removed TP? (x3): TestPoint, symbol Connector:TestPoint
- added DS1: NHD-14432WG-BTFH-V_T, User:LCD_NHD-14432WG-BTFH-V_T, symbol User:NHD-14432WG-BTFH-V_T
- added H5: MountingHole, MountingHole:MountingHole_3.2mm_M3, symbol Mechanical:MountingHole
- added R65: 56, Resistor_SMD:R_0805_2012Metric, symbol Device:R_Small
- C10, C15, C18, C30, C31, C32, C33, C34, C35, C36, C37: renamed from C?; footprint (none) -> Capacitor_SMD:C_0402_1005Metric
- C11, C14, C16, C23: renamed from C?; footprint (none) -> Capacitor_SMD:C_0805_2012Metric
- C13: renamed from C?; footprint (none) -> Capacitor_SMD:C_0402_1005Metric; Assembly (none) -> Y; LCSC Part # (none) -> C1525
- C17: renamed from C?; footprint (none) -> Capacitor_SMD:C_1206_3216Metric; Assembly (none) -> Y; LCSC Part # (none) -> C12891
- C19, C3, C5, C6, C7, C9: now fitted
- C2: footprint Capacitor_SMD:C_0603_1608Metric -> Capacitor_SMD:C_0805_2012Metric; now fitted
- C20, C22: renamed from C?; footprint (none) -> Capacitor_SMD:C_1206_3216Metric
- C21: renamed from C?; footprint (none) -> Capacitor_SMD:C_0402_1005Metric; Assembly (none) -> Y; LCSC Part # (none) -> C52923
- C25: renamed from C?; footprint Capacitor_SMD:C_0402_1005Metric -> Capacitor_SMD:C_0603_1608Metric
- D3: LCSC Part # C2290 -> C34499
- F1: renamed from F?; footprint (none) -> Fuse:Fuse_1206_3216Metric
- J1: renamed from J?; footprint (none) -> Connector_PinHeader_2.54mm:PinHeader_1x02_P2.54mm_Vertical
- J10, J11, J12, J13, J15, J16, J17, J18, J19, J20, J21, J22, J6, J7, J8: renamed from J?; footprint Eurorack:BOOMELE_PJ-320B -> User:PJ-320B
- J14: footprint Eurorack:MIDI_DIN5 -> User:MIDI_DIN5
- J2: footprint USB:USB_C_Receptacle_Amphenol_12401610E4-2A -> User:USB_C_Receptacle_Amphenol_12401610E4-2A
- J5, J9: footprint Eurorack:BOOMELE_PJ-320B -> User:PJ-320B
- R10, R11, R12, R13, R14, R15, R16, R17, R18, R19, R20, R27, R28, R29, R30, R31, R32, R33, R34, R35, R36, R37, R38, R45, R46, R47, R48, R49, R50, R51, R52, R9: renamed from R?; footprint (none) -> Resistor_SMD:R_0402_1005Metric
- R21, R22, R39, R40, R53, R54: renamed from R?; footprint (none) -> Resistor_SMD:R_0603_1608Metric; Assembly (none) -> Y; LCSC Part # (none) -> C4184
- R23, R24, R25, R26, R41, R42, R43, R44, R55, R56: renamed from R?; footprint (none) -> Resistor_SMD:R_0603_1608Metric; Assembly (none) -> Y; LCSC Part # (none) -> C21190
- R5: value 220 -> 150
- R57, R58: renamed from R?; footprint Resistor_SMD:R_0603_1608Metric -> Resistor_SMD:R_0805_2012Metric
- R63, R66: footprint Resistor_SMD:R_0603_1608Metric -> Resistor_SMD:R_0805_2012Metric
- R7: renamed from R?; footprint (none) -> Resistor_SMD:R_0603_1608Metric; Assembly (none) -> Y; LCSC Part # (none) -> C25803
- R8: renamed from R?; footprint (none) -> Resistor_SMD:R_0603_1608Metric; Assembly (none) -> Y; LCSC Part # (none) -> C22793
- SW1, SW2, SW4, SW5: footprint Button_Switch_SMD:SW_Push_1P1T_XKB_TS-1187A -> User:430182070816
- TP1, TP2, TP3, TP4, TP5, TP6, TP7, TP8: renamed from TP?; footprint (none) -> TestPoint:TestPoint_Loop_D2.50mm_Drill1.0mm
- U10, U7, U8, U9: renamed from U?; footprint (none) -> Package_SO:TSSOP-14_4.4x5mm_P0.65mm
- U6: renamed from U?; footprint (none) -> Package_SO:SOIC-8_3.9x4.9mm_P1.27mm
- gave numbers to parts that had none: 22
- renumbered Q2 to Q1
Connections:
- net UART_RX is gone; now on net UART2_RX: J1.1 (Pin_1)
- net +5V: no longer U1.5 (VBUS)
- net +5VD: now also U1.5 (VBUS), U3.3 (EN), DS1.2 (VDD), R65.1
- net BT1: now also R60.2, SW1.2, SW1.4, U4.33 (PB12); no longer R67.2, SW4.2, SW4.4, U4.53 (PC12)
- net BT2: now also U4.34 (PB13); no longer U4.52 (PC11)
- net BT3: now also R67.2, SW4.2, SW4.4, U4.35 (PB14); no longer R68.2, SW5.2, SW5.4, U4.51 (PC10)
- net ENC_CH1: now also U4.22 (PA6); no longer U4.58 (PB6)
- net ENC_CH2: now also U4.23 (PA7); no longer U4.59 (PB7)
- net GNDD: now also DS1.1 (VSS), DS1.10 (DB3), DS1.11 (DB4), DS1.12 (DB5), DS1.13 (DB6), DS1.14 (DB7), DS1.16 (LED-), DS1.7 (DB0), DS1.8 (DB1), DS1.9 (DB2)
- net SPI_MOSI: now also U4.57 (PB5), DS1.5 (R/~{W}); no longer U4.23 (PA7)
- net SPI_SCK: now also DS1.6 (E)
- net UART_TX: now also U4.53 (PC12); no longer J1.2 (Pin_2), U4.29 (PB10)
- net UART2_TX: now reaches U4.16 (PA2)
- net UART2_TX: now also J1.2 (Pin_2)
- net UART2_RX: now reaches U4.17 (PA3)
- net BT4: now reaches U4.36 (PB15)
- net BT4: now also R68.2, SW5.2, SW5.4
- net DISP_CS: now reaches U4.41 (PA8)
- net DISP_CS: now also DS1.4 (RS)
- removed net BT0: R60.2, SW1.2, SW1.4, U4.54 (PD2)
- net OLED_CSx: no longer names the net of U4.26 (PB0)
- net OLED_DC: no longer names the net of U4.25 (PC5)
- net OLED_RESx: no longer names the net of U4.24 (PC4)
- new net: DS1.15 (LED+), R65.2
- no-connect marks 46 -> 45
