File: Hardware/Kicad/Faderbay.kicad_pcb (KiCad board)
At the start: 4 copper layers, 360 x 130 mm, 168 parts, among them J1 Barrel_Jack_Switch, J14 MIDI DIN-5, J2 USB_C_Receptacle_USB2.0_14P, J3 SWD, J4 52437-2471, Q1 AO3401A, Q2 MMBT2222A, SW1 SW_Push_Dual, SW2 SW_Push_Dual, SW3 EC11E15204A3, SW4 SW_Push_Dual, SW5 SW_Push_Dual, U1 USBLC6-2SC6, U10 TL074, U2 LMR51430, U3 LMR51430, U4 STM32F405RGTx, U5 CD74HC4067M, U6 TL074, U7 TL074, U8 MCP6002, U9 TL074, Y1 16MHz

Commit message: 31/01/26
Parts:
- removed C27: 4,7u, Capacitor_SMD:C_0402_1005Metric
- removed C28, C29: 100n, Capacitor_SMD:C_0402_1005Metric
- removed J4: 52437-2471, User:524372471
- removed L1: 6.8u, Inductor_SMD:L_Changjiang_FXL0530
- removed L2: 5.6u, Inductor_SMD:L_Changjiang_FXL0630
- removed L3: 39n, Inductor_SMD:L_0402_1005Metric
- removed Q2: MMBT2222A, Package_TO_SOT_SMD:SOT-23
- removed R69: 910k, Resistor_SMD:R_0402_1005Metric
- added C30: 100n, Capacitor_SMD:C_0402_1005Metric, F.Cu at (-34.9, -132.5)
- added C31: 100n, Capacitor_SMD:C_0402_1005Metric, F.Cu at (-34.9, -130.6)
- added C32: 100n, Capacitor_SMD:C_0402_1005Metric, F.Cu at (-34.9, -128.6)
- added C33: 100n, Capacitor_SMD:C_0402_1005Metric, F.Cu at (-34.9, -126.6)
- added C34: 100n, Capacitor_SMD:C_0402_1005Metric, F.Cu at (-34.9, -124.7)
- added C35: 100n, Capacitor_SMD:C_0402_1005Metric, F.Cu at (-34.9, -122.7)
- added C36: 100n, Capacitor_SMD:C_0402_1005Metric, F.Cu at (-34.9, -120.7)
- added C37: 100n, Capacitor_SMD:C_0402_1005Metric, F.Cu at (-34.9, -118.8)
- added DS1: NHD-14432WG-BTFH-V_T, User:LCD_NHD-14432WG-BTFH-V_T, F.Cu at (-117.5, -50.2)
- added F1: 750mA, Fuse:Fuse_1206_3216Metric, F.Cu at (-30.6, -123.9)
- added FB2: 100@100MHz, Inductor_SMD:L_0805_2012Metric, F.Cu at (-23.2, -132.2)
- added FB3: 100@100MHz, Inductor_SMD:L_0805_2012Metric, F.Cu at (-23.2, -129.4)
- added H5: MountingHole, MountingHole:MountingHole_3.2mm_M3, F.Cu at (-29.5, -129.6)
- added TP1: TestPoint, TestPoint:TestPoint_Loop_D2.50mm_Drill1.0mm, F.Cu at (-52.6, -131.2)
- added TP2: TestPoint, TestPoint:TestPoint_Loop_D2.50mm_Drill1.0mm, F.Cu at (-52.6, -126.6)
- added TP3: TestPoint, TestPoint:TestPoint_Loop_D2.50mm_Drill1.0mm, F.Cu at (-48.0, -131.2)
- added TP4: TestPoint, TestPoint:TestPoint_Loop_D2.50mm_Drill1.0mm, F.Cu at (-48.0, -126.6)
- added TP5: TestPoint, TestPoint:TestPoint_Loop_D2.50mm_Drill1.0mm, F.Cu at (-43.3, -131.2)
- added TP6: TestPoint, TestPoint:TestPoint_Loop_D2.50mm_Drill1.0mm, F.Cu at (-43.3, -126.6)
- added TP7: TestPoint, TestPoint:TestPoint_Loop_D2.50mm_Drill1.0mm, F.Cu at (-38.6, -131.2)
- added TP8: TestPoint, TestPoint:TestPoint_Loop_D2.50mm_Drill1.0mm, F.Cu at (-38.6, -126.6)
- C10: value 2.2u -> 100n; footprint Capacitor_SMD:C_1206_3216Metric -> Capacitor_SMD:C_0402_1005Metric
- C11: value 2.2u -> 10u; footprint Capacitor_SMD:C_1206_3216Metric -> Capacitor_SMD:C_0805_2012Metric
- C14, C23: value 100n -> 10u; footprint Capacitor_SMD:C_0402_1005Metric -> Capacitor_SMD:C_0805_2012Metric
- C15, C18: value 22u -> 100n; footprint Capacitor_SMD:C_1206_3216Metric -> Capacitor_SMD:C_0402_1005Metric
- C16: value 22u -> 10u; footprint Capacitor_SMD:C_1206_3216Metric -> Capacitor_SMD:C_0805_2012Metric
- C17: value 22u -> 100u
- C2: footprint Capacitor_SMD:C_0603_1608Metric -> Capacitor_SMD:C_0805_2012Metric
- C20: value 100n -> 100u; footprint Capacitor_SMD:C_0402_1005Metric -> Capacitor_SMD:C_1206_3216Metric
- C21: value 1u -> 100n
- C22: value 10n -> 10u; footprint Capacitor_SMD:C_0402_1005Metric -> Capacitor_SMD:C_1206_3216Metric
- C25: value 100n -> 10u; footprint Capacitor_SMD:C_0402_1005Metric -> Capacitor_SMD:C_0603_1608Metric
- C26: value 100n -> 10n
- FB1: value 600 @ 6600MHz -> 100@100MHz
- J1: value Barrel_Jack_Switch -> UART; footprint Connector_BarrelJack:BarrelJack_Kycon_KLDX-0202-xC_Horizontal -> Connector_PinHeader_2.54mm:PinHeader_1x02_P2.54mm_Vertical
- J10, J11, J12, J13, J15, J16, J17, J18, J19, J20, J21, J22, J5, J6, J7, J8, J9: footprint Eurorack:BOOMELE_PJ-320B -> User:PJ-320B
- J14: footprint Eurorack:MIDI_DIN5 -> User:MIDI_DIN5
- J2: footprint USB:USB_C_Receptacle_Amphenol_12401610E4-2A -> User:USB_C_Receptacle_Amphenol_12401610E4-2A
- Q1: value AO3401A -> MMBT2222A
- R10: value 22.1k -> 10k; footprint Resistor_SMD:R_0603_1608Metric -> Resistor_SMD:R_0402_1005Metric
- R11, R12, R13, R14, R15, R16, R29, R30, R31, R32, R33, R34, R47, R48, R49, R50: footprint Resistor_SMD:R_0603_1608Metric -> Resistor_SMD:R_0402_1005Metric
- R17, R18, R19, R20, R35, R36, R37, R38, R51, R52: value 20k -> 10k; footprint Resistor_SMD:R_0603_1608Metric -> Resistor_SMD:R_0402_1005Metric
- R21, R22, R39, R40, R53, R54: value 20k -> 1k
- R27, R28, R45, R46: value 1k -> 10k; footprint Resistor_SMD:R_0603_1608Metric -> Resistor_SMD:R_0402_1005Metric
- R4: value 560 -> 230
- R5: value 220 -> 150
- R57, R58: value 1k -> 220; footprint Resistor_SMD:R_0603_1608Metric -> Resistor_SMD:R_0805_2012Metric
- R63, R66: footprint Resistor_SMD:R_0603_1608Metric -> Resistor_SMD:R_0805_2012Metric
- R64: value 10k -> 1k
- R65: value 10k -> 56; footprint Resistor_SMD:R_0402_1005Metric -> Resistor_SMD:R_0805_2012Metric
- R7: value 100k -> 0
- R8: value 13.7k -> 0
- R9: value 100k -> 10k; footprint Resistor_SMD:R_0603_1608Metric -> Resistor_SMD:R_0402_1005Metric
- RV1, RV10, RV11, RV12, RV13, RV14, RV15, RV16, RV2, RV3, RV4, RV5, RV6, RV7, RV8, RV9: value R_Potentiometer -> 100k
- SW1, SW2, SW4, SW5: footprint Button_Switch_SMD:SW_Push_1P1T_XKB_TS-1187A -> User:430182070816
- U10, U7, U9: value TL074 -> MCP6004; footprint Package_SO:SOIC-14_3.9x8.7mm_P1.27mm -> Package_SO:TSSOP-14_4.4x5mm_P0.65mm
- U2: value LMR51430 -> MCP6001-OT; footprint Package_TO_SOT_SMD:SOT-23-6 -> Package_TO_SOT_SMD:SOT-23-5
- U3: value LMR51430 -> TLV75733PDBV; footprint Package_TO_SOT_SMD:SOT-23-6 -> Package_TO_SOT_SMD:SOT-23-5
- U6: value TL074 -> ICL7660; footprint Package_SO:SOIC-14_3.9x8.7mm_P1.27mm -> Package_SO:SOIC-8_3.9x4.9mm_P1.27mm
- U8: value MCP6002 -> MCP6004; footprint Package_SO:SOIC-8_3.9x4.9mm_P1.27mm -> Package_SO:TSSOP-14_4.4x5mm_P0.65mm
Connections:
- net J2 renamed Net-(J7-Pad3)
- net J3 renamed Net-(J8-Pad3)
- net J4 renamed Net-(J10-Pad3)
- net J5 renamed Net-(J11-Pad3)
- C1 pad 2: GND -> GNDD
- C10 pad 1: GND -> +3.3V
- C10 pad 2: +12V -> GNDD
- C11 pad 1: GND -> +5VD
- C11 pad 2: +12V -> GNDD
- C12 pad 2: GND -> GNDD
- C13 pad 1: Net-(U2-SW) -> +5VD
- C13 pad 2: Net-(U2-CB) -> GNDD
- C14 pad 1: Net-(U3-SW) -> +3.3V
- C14 pad 2: Net-(U3-CB) -> GNDD
- C15 pad 1: GND -> +3.3V
- C15 pad 2: +5V -> GNDD
- C16 pad 1: GND -> +5VA
- C16 pad 2: +3.3V -> GNDA
- C17 pad 1: GND -> +5VA
- C17 pad 2: +5V -> GNDA
- C18 pad 1: GND -> +5VA
- C18 pad 2: +3.3V -> GNDA
- C2 pad 2: GND -> GNDD
- C20 pad 1: +3.3V -> +5VD
- C20 pad 2: GND -> GNDD
- C21 pad 1: Net-(U8A-+) -> +5VD
- C21 pad 2: GND -> GNDD
- C22 pad 1: Net-(U8A-+) -> Net-(U6-CAP+)
- C22 pad 2: GND -> Net-(U6-CAP-)
- C23 pad 1: +12V -> -5VA
- C23 pad 2: GND -> GNDA
- C24 pad 1: +12V -> Net-(C24-Pad1)
- C24 pad 2: GND -> GNDA
- C25 pad 1: +12V -> Net-(C24-Pad1)
- C25 pad 2: GND -> VDDA
- C26 pad 1: +12V -> VDDA
- C26 pad 2: GND -> GNDA
- C3 pad 2: GND -> GNDD
- C4 pad 2: GND -> GNDD
- C5 pad 2: GND -> GNDD
- C6 pad 2: GND -> GNDD
- C7 pad 2: GND -> GNDD
- C8 pad 2: GND -> GNDD
- C9 pad 2: GND -> GNDD
- D2 pad 1: GND -> GNDD
- D3 pad 1: GND -> GNDD
- FB1 pad 1: Net-(Q1-S) -> +5VD
- FB1 pad 2: +12V -> +5VA
- J1 pad 1: Net-(S1-NO_1) -> UART2_RX
- J1 pad 2: Net-(S1-NO_2) -> UART2_TX
- J10 pad 1: GND -> GNDA
- J10 pad 2: GND -> GNDA
- J11 pad 1: GND -> GNDA
- J11 pad 2: GND -> GNDA
- J12 pad 1: GND -> GNDA
- J12 pad 2: GND -> GNDA
- J12 pad 3: J6 -> Net-(J12-Pad3)
- J13 pad 1: GND -> GNDA
- J13 pad 2: GND -> GNDA
- J13 pad 3: J7 -> Net-(J13-Pad3)
- J14 pad 2: GND -> unconnected-(J14-Pad2)
- J14 pad 4: MIDI_TRS_R -> Net-(J14-Pad4)
- J14 pad 5: MIDI_TRS_T -> Net-(J14-Pad5)
- J15 pad 1: GND -> GNDA
- J15 pad 2: GND -> GNDA
- J15 pad 3: J8 -> Net-(J15-Pad3)
- J16 pad 1: GND -> GNDA
- J16 pad 2: GND -> GNDA
- J16 pad 3: J9 -> Net-(J16-Pad3)
- J17 pad 1: GND -> GNDA
- J17 pad 2: GND -> GNDA
- J17 pad 3: J10 -> Net-(J17-Pad3)
- J18 pad 1: GND -> GNDA
- J18 pad 2: GND -> GNDA
- J18 pad 3: J11 -> Net-(J18-Pad3)
- J19 pad 1: GND -> GNDA
- J19 pad 2: GND -> GNDA
- J19 pad 3: J12 -> Net-(J19-Pad3)
- J2 pad A4: USB_VBUS -> Net-(F1-Pad1)
- J2 pad A9: USB_VBUS -> Net-(F1-Pad1)
- J2 pad B4: USB_VBUS -> Net-(F1-Pad1)
- J2 pad B9: USB_VBUS -> Net-(F1-Pad1)
- J20 pad 1: GND -> GNDA
- J20 pad 2: GND -> GNDA
- J20 pad 3: J13 -> Net-(J20-Pad3)
- J21 pad 1: GND -> GNDA
- J21 pad 2: GND -> GNDA
- J21 pad 3: J14 -> Net-(J21-Pad3)
- J22 pad 1: GND -> GNDA
- J22 pad 2: GND -> GNDA
- J22 pad 3: J15 -> Net-(J22-Pad3)
- J3 pad 3: GND -> GNDD
- J3 pad 5: GND -> GNDD
- J3 pad 9: GND -> GNDD
- J5 pad 1: GND -> GNDA
- J5 pad 2: GND -> GNDA
- J5 pad 3: J0 -> Net-(J5-Pad3)
- J6 pad 1: GND -> GNDA
- J6 pad 2: GND -> GNDA
- J6 pad 3: J1 -> Net-(J6-Pad3)
- J7 pad 1: GND -> GNDA
- J7 pad 2: GND -> GNDA
- J8 pad 1: GND -> GNDA
- J8 pad 2: GND -> GNDA
- J9 pad 1: GND -> GNDD
- J9 pad 2: MIDI_TRS_R -> Net-(J9-Pad2)
- J9 pad 3: MIDI_TRS_T -> Net-(J9-Pad3)
- Q1 pad 1: GND -> Net-(Q1-B)
- Q1 pad 2: Net-(Q1-S) -> GNDD
- Q1 pad 3: 12V_In -> Net-(Q1-C)
- R10 pad 1: GND -> +5VA
- R10 pad 2: Net-(U3-FB) -> Net-(U7B--)
- R11 pad 1: Net-(U6C--) -> +5VA
- R11 pad 2: GND -> Net-(U7C--)
- R12 pad 1: Net-(U6D--) -> +5VA
- R12 pad 2: GND -> Net-(U7D--)
- R13 pad 2: GND -> Net-(R13-Pad2)
- R14 pad 2: GND -> Net-(R14-Pad2)
- R15 pad 1: Net-(U6A--) -> Net-(U7C--)
- R15 pad 2: GND -> Net-(R15-Pad2)
- R16 pad 1: Net-(U6B--) -> Net-(U7D--)
- R16 pad 2: GND -> Net-(R16-Pad2)
- R17 pad 1: Net-(U6C--) -> +5VA
- R17 pad 2: Net-(R17-Pad2) -> Net-(U8A--)
- R18 pad 1: Net-(U6D--) -> +5VA
- R18 pad 2: Net-(R18-Pad2) -> Net-(U8B--)
- R19 pad 1: Net-(U7A--) -> Net-(U8A--)
- R20 pad 1: Net-(U7B--) -> Net-(U8B--)
- R21 pad 1: Net-(U6A--) -> Net-(R13-Pad2)
- R21 pad 2: Net-(R21-Pad2) -> Net-(J5-Pad3)
- R22 pad 1: Net-(U6B--) -> Net-(R14-Pad2)
- R22 pad 2: Net-(R22-Pad2) -> Net-(J6-Pad3)
- R23 pad 1: Net-(R17-Pad2) -> Net-(R15-Pad2)
- R24 pad 1: Net-(R18-Pad2) -> Net-(R16-Pad2)
- R27 pad 1: Net-(R21-Pad2) -> +5VA
- R27 pad 2: J0 -> Net-(U9A--)
- R28 pad 1: Net-(R22-Pad2) -> +5VA
- R28 pad 2: J1 -> Net-(U9B--)
- R29 pad 1: Net-(U9D--) -> +5VA
- R29 pad 2: GND -> Net-(U8C--)
- R30 pad 1: Net-(U7C--) -> +5VA
- R30 pad 2: GND -> Net-(U8D--)
- R31 pad 1: Net-(U7D--) -> +5VA
- R31 pad 2: GND -> Net-(U9C--)
- R32 pad 1: Net-(U9A--) -> +5VA
- R32 pad 2: GND -> Net-(U9D--)
- R33 pad 1: Net-(U9B--) -> Net-(U9A--)
- R33 pad 2: GND -> Net-(R33-Pad2)
- R34 pad 1: Net-(U9C--) -> Net-(U9B--)
- R34 pad 2: GND -> Net-(R34-Pad2)
- R35 pad 1: Net-(U9D--) -> Net-(U8C--)
- R36 pad 1: Net-(U7C--) -> Net-(U8D--)
- R37 pad 1: Net-(U7D--) -> Net-(U9C--)
- R38 pad 1: Net-(U9A--) -> Net-(U9D--)
- R39 pad 1: Net-(U9B--) -> Net-(R33-Pad2)
- R39 pad 2: Net-(R39-Pad2) -> Net-(J12-Pad3)
- R4 pad 2: +12V -> +5V
- R40 pad 1: Net-(U9C--) -> Net-(R34-Pad2)
- R40 pad 2: Net-(R40-Pad2) -> Net-(J13-Pad3)
- R41 pad 2: J11 -> Net-(J15-Pad3)
- R42 pad 2: J6 -> Net-(J16-Pad3)
- R43 pad 2: J7 -> Net-(J17-Pad3)
- R44 pad 2: J8 -> Net-(J18-Pad3)
- R45 pad 1: Net-(R39-Pad2) -> +5VA
- R45 pad 2: J9 -> Net-(U10A--)
- R46 pad 1: Net-(R40-Pad2) -> +5VA
- R46 pad 2: J10 -> Net-(U10B--)
- R47 pad 1: Net-(U10A--) -> +5VA
- R47 pad 2: GND -> Net-(U10C--)
- R48 pad 1: Net-(U10B--) -> +5VA
- R48 pad 2: GND -> Net-(U10D--)
- R49 pad 1: Net-(U10C--) -> Net-(U10A--)
- R49 pad 2: GND -> Net-(R49-Pad2)
- R50 pad 1: Net-(U10D--) -> Net-(U10B--)
- R50 pad 2: GND -> Net-(R50-Pad2)
- R51 pad 1: Net-(U10A--) -> Net-(U10C--)
- R52 pad 1: Net-(U10B--) -> Net-(U10D--)
- R53 pad 1: Net-(U10C--) -> Net-(R49-Pad2)
- R53 pad 2: Net-(R53-Pad2) -> Net-(J19-Pad3)
- R54 pad 1: Net-(U10D--) -> Net-(R50-Pad2)
- R54 pad 2: Net-(R54-Pad2) -> Net-(J20-Pad3)
- R55 pad 2: J12 -> Net-(J21-Pad3)
- R56 pad 2: J13 -> Net-(J22-Pad3)
- R57 pad 1: Net-(R53-Pad2) -> Net-(Q1-C)
- R57 pad 2: J14 -> Net-(J9-Pad3)
- R58 pad 1: Net-(R54-Pad2) -> +5V
- R58 pad 2: J15 -> Net-(J9-Pad2)
- R60 pad 1: GND -> GNDD
- R60 pad 2: BT0 -> BT1
- R61 pad 1: GND -> GNDD
- R63 pad 1: MIDI_TRS_R -> Net-(J14-Pad4)
- R64 pad 1: Net-(Q2-B) -> Net-(Q1-B)
- R65 pad 1: +5V -> +5VD
- R65 pad 2: MIDI_OUT -> Net-(DS1-LED+)
- R66 pad 1: MIDI_OUT -> Net-(Q1-C)
- R66 pad 2: MIDI_TRS_T -> Net-(J14-Pad5)
- R67 pad 1: GND -> GNDD
- R67 pad 2: BT1 -> BT3
- R68 pad 1: GND -> GNDD
- R68 pad 2: BT3 -> BT4
- R7 pad 1: Net-(U2-FB) -> GND
- R7 pad 2: +5V -> GNDD
- R8 pad 2: Net-(U2-FB) -> GNDA
- R9 pad 1: Net-(U3-FB) -> +5VA
- R9 pad 2: +3.3V -> Net-(U7A--)
- RV1 pad 1: VDDA -> +5VA
- RV1 pad 3: GND -> GNDA
- RV10 pad 1: VDDA -> +5VA
- RV10 pad 2: P9 -> P7
- RV10 pad 3: GND -> GNDA
- RV11 pad 1: VDDA -> +5VA
- RV11 pad 2: P10 -> P14
- RV11 pad 3: GND -> GNDA
- RV12 pad 1: VDDA -> +5VA
- RV12 pad 2: P11 -> P15
- RV12 pad 3: GND -> GNDA
- RV13 pad 1: VDDA -> +5VA
- RV13 pad 2: P12 -> P8
- RV13 pad 3: GND -> GNDA
- RV14 pad 1: VDDA -> +5VA
- RV14 pad 2: P13 -> P9
- RV14 pad 3: GND -> GNDA
- RV15 pad 1: VDDA -> +5VA
- RV15 pad 2: P14 -> P10
- RV15 pad 3: GND -> GNDA
- RV16 pad 1: VDDA -> +5VA
- RV16 pad 2: P15 -> P11
- RV16 pad 3: GND -> GNDA
- RV2 pad 1: VDDA -> +5VA
- RV2 pad 3: GND -> GNDA
- RV3 pad 1: VDDA -> +5VA
- RV3 pad 3: GND -> GNDA
- RV4 pad 1: VDDA -> +5VA
- RV4 pad 3: GND -> GNDA
- RV5 pad 1: VDDA -> +5VA
- RV5 pad 2: P4 -> P12
- RV5 pad 3: GND -> GNDA
- RV6 pad 1: VDDA -> +5VA
- RV6 pad 2: P5 -> P13
- RV6 pad 3: GND -> GNDA
- RV7 pad 1: VDDA -> +5VA
- RV7 pad 2: P6 -> P4
- RV7 pad 3: GND -> GNDA
- RV8 pad 1: VDDA -> +5VA
- RV8 pad 2: P7 -> P5
- RV8 pad 3: GND -> GNDA
- RV9 pad 1: VDDA -> +5VA
- RV9 pad 2: P8 -> P6
- RV9 pad 3: GND -> GNDA
- S1 pad 1: Net-(S1-NO_1) -> +5VD
- S1 pad 2: 12V_In -> Net-(S1-COM_1)
- S1 pad 5: GND -> unconnected-(S1-COM_2-Pad5)
- S1 pad 6: Net-(S1-NO_2) -> unconnected-(S1-NO_2-Pad6)
- S1 pad MH1: GND -> unconnected-(S1-PadMH1)
- S1 pad MH2: GND -> unconnected-(S1-PadMH2)
- SW1 pad 2: BT0 -> BT1
- SW3 pad C1: GND -> GNDD
- SW3 pad MH1: GND -> GNDD
- SW3 pad MH2: GND -> GNDD
- SW4 pad 2: BT1 -> BT3
- SW5 pad 2: BT3 -> BT4
- U1 pad 2: GND -> GNDD
- U1 pad 5: +5V -> +5VD
- U10 pad 1: Net-(R51-Pad2) -> Net-(R49-Pad2)
- U10 pad 10: P14 -> P10
- U10 pad 11: GND -> -5VA
- U10 pad 12: P15 -> P11
- U10 pad 14: Net-(R54-Pad2) -> Net-(R52-Pad2)
- U10 pad 3: P12 -> P8
- U10 pad 4: +12V -> +5VA
- U10 pad 5: P13 -> P9
- U10 pad 7: Net-(R52-Pad2) -> Net-(R50-Pad2)
- U10 pad 8: Net-(R53-Pad2) -> Net-(R51-Pad2)
- U2 pad 1: GND -> ADC_IN
- U2 pad 2: Net-(U2-SW) -> +3.3V
- U2 pad 3: +12V -> ADC_BUFF
- U2 pad 4: Net-(U2-FB) -> ADC_IN
- U2 pad 5: +12V -> GNDD
- U3 pad 1: GND -> +5VD
- U3 pad 2: Net-(U3-SW) -> GNDD
- U3 pad 3: +12V -> +5VD
- U3 pad 4: Net-(U3-FB) -> unconnected-(U3-NC-Pad4)
- U3 pad 5: +12V -> +3.3V
- U4 pad 12: GND -> GNDA
- U4 pad 16: unconnected-(U4-PA2-Pad16) -> UART2_TX
- U4 pad 17: unconnected-(U4-PA3-Pad17) -> UART2_RX
- U4 pad 18: GND -> GNDD
- U4 pad 22: unconnected-(U4-PA6-Pad22) -> ENC_CH1
- U4 pad 23: SPI_MOSI -> ENC_CH2
- U4 pad 24: OLED_RESx -> unconnected-(U4-PC4-Pad24)
- U4 pad 25: OLED_DC -> unconnected-(U4-PC5-Pad25)
- U4 pad 26: OLED_CSx -> unconnected-(U4-PB0-Pad26)
- U4 pad 29: UART_TX -> unconnected-(U4-PB10-Pad29)
- U4 pad 33: unconnected-(U4-PB12-Pad33) -> BT1
- U4 pad 34: unconnected-(U4-PB13-Pad34) -> BT2
- U4 pad 35: unconnected-(U4-PB14-Pad35) -> BT3
- U4 pad 36: unconnected-(U4-PB15-Pad36) -> BT4
- U4 pad 41: unconnected-(U4-PA8-Pad41) -> DISP_CS
- U4 pad 51: BT3 -> unconnected-(U4-PC10-Pad51)
- U4 pad 52: BT2 -> unconnected-(U4-PC11-Pad52)
- U4 pad 53: BT1 -> UART_TX
- U4 pad 54: BT0 -> unconnected-(U4-PD2-Pad54)
- U4 pad 57: unconnected-(U4-PB5-Pad57) -> SPI_MOSI
- U4 pad 58: ENC_CH1 -> unconnected-(U4-PB6-Pad58)
- U4 pad 59: ENC_CH2 -> unconnected-(U4-PB7-Pad59)
- U4 pad 60: GND -> GNDD
- U4 pad 63: GND -> GNDD
- U5 pad 12: GND -> GNDD
- U6 pad 1: Net-(R21-Pad2) -> unconnected-(U6-NC-Pad1)
- U6 pad 2: Net-(U6A--) -> Net-(U6-CAP+)
- U6 pad 3: P0 -> GNDA
- U6 pad 4: +12V -> Net-(U6-CAP-)
- U6 pad 5: P1 -> Net-(U6-VOUT)
- U6 pad 6: Net-(U6B--) -> unconnected-(U6-LV-Pad6)
- U6 pad 7: Net-(R22-Pad2) -> +5VA
- U6 pad 8: Net-(R17-Pad2) -> +5VA
- U7 pad 1: Net-(R19-Pad2) -> Net-(R13-Pad2)
- U7 pad 10: P6 -> P2
- U7 pad 11: GND -> -5VA
- U7 pad 12: P7 -> P3
- U7 pad 14: Net-(R37-Pad2) -> Net-(R16-Pad2)
- U7 pad 3: P4 -> P0
- U7 pad 4: +12V -> +5VA
- U7 pad 5: P5 -> P1
- U7 pad 7: Net-(R20-Pad2) -> Net-(R14-Pad2)
- U7 pad 8: Net-(R36-Pad2) -> Net-(R15-Pad2)
- U8 pad 1: VDDA -> Net-(R19-Pad2)
- U8 pad 2: VDDA -> Net-(U8A--)
- U8 pad 3: Net-(U8A-+) -> P12
- U8 pad 4: GND -> +5VA
- U8 pad 5: ADC_BUFF -> P13
- U8 pad 6: ADC_IN -> Net-(U8B--)
- U8 pad 7: ADC_IN -> Net-(R20-Pad2)
- U8 pad 8: +3.3V -> Net-(R35-Pad2)
- U9 pad 1: Net-(R38-Pad2) -> Net-(R33-Pad2)
- U9 pad 10: P10 -> P14
- U9 pad 11: GND -> -5VA
- U9 pad 12: P11 -> P15
- U9 pad 14: Net-(R35-Pad2) -> Net-(R38-Pad2)
- U9 pad 3: P8 -> P4
- U9 pad 4: +12V -> +5VA
- U9 pad 5: P9 -> P5
- U9 pad 7: Net-(R39-Pad2) -> Net-(R34-Pad2)
- U9 pad 8: Net-(R40-Pad2) -> Net-(R37-Pad2)
- Y1 pad 2: GND -> GNDD
- Y1 pad 4: GND -> GNDD
Routing:
- net +12V: track 483.5 -> 0.00 mm, vias 12 -> 0
- net GND: track 417.2 -> 0.00 mm, vias 72 -> 0
- net +3.3V: track 292.9 -> 0.00 mm, vias 18 -> 0
- net OLED_DC: track 214.5 -> 0.00 mm, vias 4 -> 0
- net SPI_MOSI: track 213.8 -> 0.00 mm, vias 2 -> 0
- net OLED_RESx: track 213.1 -> 0.00 mm, vias 4 -> 0
- net OLED_CSx: track 212.6 -> 0.00 mm, vias 4 -> 0
- net SPI_SCK: track 211.9 -> 0.00 mm, vias 2 -> 0
- net P15: track 204.6 -> 0.00 mm, vias 3 -> 0
- net P14: track 191.6 -> 0.00 mm, vias 3 -> 0
- net P12: track 184.7 -> 0.00 mm, vias 3 -> 0
- net P0: track 181.3 -> 0.00 mm, vias 2 -> 0
- net P13: track 174.9 -> 0.00 mm, vias 3 -> 0
- net P1: track 158.5 -> 0.00 mm, vias 2 -> 0
- net P11: track 154.6 -> 0.00 mm, vias 4 -> 0
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- removed copper zone on In2.Cu, net +12V
Other:
- board size 360 x 130 mm -> 360 x 140 mm

Commit message: Update hardware: KiCad, Gerbers, BOM, new schematic variants
Parts:
- removed D3: WHITE, LED_SMD:LED_0603_1608Metric
- removed the G*** at (-134.9, -49.5)
- removed the H1 at (-174.1, -59.6)
- removed J14: MIDI DIN-5, User:MIDI_DIN5
- removed R6: 220, Resistor_SMD:R_0603_1608Metric
- removed R63, R66: 220, Resistor_SMD:R_0805_2012Metric
- removed S1: LC2255EENPTAGBLK, User:LC2255EENPTAGBLK
- added C27: 100n, Capacitor_SMD:C_0402_1005Metric, F.Cu at (-169.2, -19.3)
- added C38: 100n, Capacitor_SMD:C_0402_1005Metric, F.Cu at (33.2, -41.8)
- added FID1: Fiducial_1mm_Mask2mm, Fiducial:Fiducial_1mm_Mask2mm, F.Cu at (-176.2, 51.8)
- added FID2: Fiducial_1mm_Mask2mm, Fiducial:Fiducial_1mm_Mask2mm, F.Cu at (176.8, 51.5)
- added FID3: Fiducial_1mm_Mask2mm, Fiducial:Fiducial_1mm_Mask2mm, F.Cu at (177.5, -60.2)
- added R69: 33k, Resistor_SMD:R_0402_1005Metric, F.Cu at (25.0, -36.5)
- added R70: 56k, Resistor_SMD:R_0402_1005Metric, F.Cu at (28.0, -37.8)
- added R71: 10k, Capacitor_SMD:C_0402_1005Metric, F.Cu at (39.2, -50.8)
- added SW6: SW_SPST, footprints:RA1H1C112R, F.Cu at (159.5, -59.0)
- added U11: 74AHCT125, Package_SO:SOIC-14_3.9x8.7mm_P1.27mm, F.Cu at (-173.8, -16.0)
- D1: footprint User:WP934EWGD -> footprints:WP934EWGD
- DS1: footprint User:LCD_NHD-14432WG-BTFH-V_T -> footprints:LCD_NHD-14432WG-BTFH-V_T
- J10, J11, J12, J13, J15, J16, J17, J18, J19, J20, J21, J22, J5, J6, J7, J8, J9: footprint User:PJ-320B -> footprints:PJ-320B
- J2: footprint User:USB_C_Receptacle_Amphenol_12401610E4-2A -> User:USB_C_Receptacle_HRO_TYPE-C-31-M-12
- R4: value 230 -> 220
- RV1, RV10, RV11, RV12, RV13, RV14, RV15, RV16, RV2, RV3, RV4, RV5, RV6, RV7, RV8, RV9: footprint User:PTB60442010BPA104 -> Potentiometer_THT:Potentiometer_Bourns_PTA6043_Single_Slide
- SW1, SW2, SW4, SW5: footprint User:430182070816 -> footprints:430182070816
- SW3: footprint User:EC11E15204A3 -> footprints:EC11E15204A3
- moved R65 270.6 mm to (-148.6, -71.0), turned to 0 degrees
- moved U6 266.2 mm to (169.5, -35.9)
- moved TP7 257.4 mm to (172.5, 16.0)
- moved TP5 256.3 mm to (172.5, 7.00)
- moved TP6 256.2 mm to (172.5, 11.5)
- moved TP3 255.5 mm to (172.5, -2.00)
- moved TP4 255.4 mm to (172.5, 2.50)
- moved TP1 255.2 mm to (172.5, -11.0)
- moved TP2 255.1 mm to (172.5, -6.50)
- moved C23 250.3 mm to (172.1, -31.5)
- moved R9 239.3 mm to (-85.0, -36.5), turned to 90 degrees
- moved R10 234.7 mm to (-80.5, -36.5), turned to 90 degrees
- moved FB2 222.3 mm to (175.5, -32.4), turned to -90 degrees
- moved C24 217.0 mm to (115.5, -39.0), turned to -90 degrees
- moved F1 183.7 mm to (144.5, -68.5)
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- renumbered H2 to H1, H3 to H2, H4 to H3, H5 to H4
Connections:
- C19 pad 1: GND -> GNDD
- DS1 pad 4: DISP_CS -> ~CS
- DS1 pad 5: SPI_MOSI -> SID
- DS1 pad 6: SPI_SCK -> SCLK
- DS1 pad S1: unconnected-(DS1-SHIELD-PadS1) -> GNDD
- DS1 pad S2: unconnected-(DS1-SHIELD__1-PadS2) -> GNDD
- DS1 pad S3: unconnected-(DS1-SHIELD__2-PadS3) -> GNDD
- DS1 pad S4: unconnected-(DS1-SHIELD__3-PadS4) -> GNDD
- R4 pad 2: +5V -> +5VD
- R58 pad 1: +5V -> +5VD
- RV10 pad 2: P7 -> P9
- RV11 pad 2: P14 -> P10
- RV12 pad 2: P15 -> P11
- RV13 pad 2: P8 -> P12
- RV14 pad 2: P9 -> P13
- RV15 pad 2: P10 -> P14
- RV16 pad 2: P11 -> P15
- RV5 pad 2: P12 -> P4
- RV6 pad 2: P13 -> P5
- RV7 pad 2: P4 -> P6
- RV8 pad 2: P5 -> P7
- RV9 pad 2: P6 -> P8
- U10 pad 10: P10 -> P14
- U10 pad 12: P11 -> P15
- U10 pad 3: P8 -> P12
- U10 pad 5: P9 -> P13
- U2 pad 2: +3.3V -> GNDD
- U2 pad 3: ADC_BUFF -> Net-(U2-+)
- U2 pad 5: GNDD -> +3.3V
- U4 pad 60: GNDD -> Net-(U4-BOOT0)
- U5 pad 15: GND -> GNDD
- U8 pad 10: P6 -> P8
- U8 pad 12: P7 -> P9
- U8 pad 3: P12 -> P4
- U8 pad 5: P13 -> P5
- U9 pad 10: P14 -> P10
- U9 pad 12: P15 -> P11
- U9 pad 3: P4 -> P6
- U9 pad 5: P5 -> P7
Routing:
- net GNDA: track 0.00 -> 822.7 mm, vias 0 -> 29
- net +5VA: track 0.00 -> 579.5 mm, vias 0 -> 23
- net +5VD: track 0.00 -> 539.5 mm, vias 0 -> 7
- net -5VA: track 0.00 -> 347.0 mm, vias 0 -> 3
- net +3.3V: track 0.00 -> 302.3 mm, vias 0 -> 13
- net SPI_MOSI: track 0.00 -> 257.6 mm, vias 0 -> 2
- net SPI_SCK: track 0.00 -> 249.8 mm, vias 0 -> 2
- net DISP_CS: track 0.00 -> 242.7 mm, vias 0 -> 2
- net P15: track 0.00 -> 237.0 mm, vias 0 -> 9
- net P14: track 0.00 -> 213.1 mm, vias 0 -> 3
- net P13: track 0.00 -> 193.6 mm, vias 0 -> 4
- net VDDA: track 0.00 -> 173.6 mm, vias 0 -> 1
- net P9: track 0.00 -> 156.5 mm, vias 0 -> 5
- net P12: track 0.00 -> 155.5 mm, vias 0 -> 2
- net P0: track 0.00 -> 152.0 mm, vias 0 -> 1
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- added copper zone on F.Cu, net +3.3V
- added copper zone on F.Cu, net +5VA
- added copper zone on F.Cu, net GNDA
- added copper zone on F.Cu, net GNDD
- added copper zone on In1.Cu, net GNDD
- removed copper zone on In2.Cu, net +3.3V
- removed copper zone on In2.Cu, net +5V
- removed copper zone on In1.Cu, net GND
- removed copper zone on In2.Cu, net VDDA
Other:
- board text added: "Designed by VonMartins v0.1 - 2026/05/11"
- board text added: "UART"
- board text removed: "Designed by Marti Dominguez Rev. 1.0 25-04-2025"
