File: Hardware/Kicad/Faderbay_MidiDin5.kicad_sch (KiCad schematic)
At the start: 178 parts, among them J1 UART, J2 USB_C_Receptacle_USB2.0_14P, J3 SWD, Q1 MMBT2222A, SW1 SW_Push_Dual, SW2 SW_Push_Dual, SW3 EC11E15204A3, SW4 SW_Push_Dual, SW5 SW_Push_Dual, SW6 SW_SPST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

Commit message: Update hardware: KiCad, Gerbers, BOM, new schematic variants
Parts:
- removed C27, C38: 100n, Capacitor_SMD:C_0402_1005Metric, symbol Device:C_Small
- removed R69: 33k, Resistor_SMD:R_0402_1005Metric, symbol Device:R_Small
- removed R70: 56k, Resistor_SMD:R_0402_1005Metric, symbol Device:R_Small
- removed R71: 10k, Capacitor_SMD:C_0402_1005Metric, symbol Device:R_Small
- removed SW6: SW_SPST, footprints:RA1H1C112R, symbol Switch:SW_SPST
- removed U11: 74AHCT125, Package_SO:SOIC-14_3.9x8.7mm_P1.27mm, symbol 74xx:74AHCT125
- added D3: WHITE, LED_SMD:LED_0603_1608Metric, symbol Device:LED
- added H1: MountingHole, MountingHole:MountingHole_3.2mm_M3, symbol Mechanical:MountingHole
- added J14: MIDI DIN-5, footprints:MIDI_DIN5, symbol Eurorack:MIDI DIN-5
- added R6: 220, Resistor_SMD:R_0603_1608Metric, symbol Device:R_Small
- added R63, R66: 220, Resistor_SMD:R_0805_2012Metric, symbol Device:R_Small
- added S1: LC2255EENPTAGBLK, footprints:LC2255EENPTAGBLK, symbol User:LC2255EENPTAGBLK
- J10, J11, J12, J13, J15, J16, J17, J18, J19, J20, J21, J22, J5, J6, J7, J8, J9: value (none) -> ~
- J2: footprint User:USB_C_Receptacle_HRO_TYPE-C-31-M-12 -> footprints:USB_C_Receptacle_Amphenol_12401610E4-2A
- R4: value 220 -> 230
- RV1, RV10, RV11, RV12, RV13, RV14, RV15, RV16, RV2, RV3, RV4, RV5, RV6, RV7, RV8, RV9: footprint Potentiometer_THT:Potentiometer_Bourns_PTA6043_Single_Slide -> footprints:PTB60442010BPA104
- renumbered H1 to H2, H2 to H3, H3 to H4, H4 to H5
Connections:
- net SCLK is gone; now on net SPI_SCK: DS1.6 (E)
- net SID is gone; now on net SPI_MOSI: DS1.5 (R/~{W})
- net ~CS is gone; now on net DISP_CS: DS1.4 (RS)
- net +3.3V: now also U2.2 (V-); no longer U2.5 (V+)
- net +5VD: now also S1.1 (NO_1); no longer R4.2, R58.1
- net ADC_BUFF: now also U2.3 (+)
- net GND: now also C19.1, U5.15 (~{E})
- net GNDD: now also U2.5 (V+), U4.60 (BOOT0), D3.1 (K); no longer C19.1, DS1.S1 (SHIELD), DS1.S2 (SHIELD__1), DS1.S3 (SHIELD__2), DS1.S4 (SHIELD__3), U2.2 (V-), U5.15 (~{E})
- net P10: now also RV15.2, U10.10 (+); no longer RV11.2, U9.10 (+)
- net P11: now also RV16.2, U10.12 (+); no longer RV12.2, U9.12 (+)
- net P12: now also RV5.2, U8.3 (+); no longer RV13.2, U10.3 (+)
- net P13: now also RV6.2, U8.5 (+); no longer RV14.2, U10.5 (+)
- net P14: now also RV11.2, U9.10 (+); no longer RV15.2, U10.10 (+)
- net P15: now also RV12.2, U9.12 (+); no longer RV16.2, U10.12 (+)
- net P4: now also RV7.2, U9.3 (+); no longer RV5.2, U8.3 (+)
- net P5: now also RV8.2, U9.5 (+); no longer RV6.2, U8.5 (+)
- net P6: now also RV9.2, U8.10 (+); no longer RV7.2, U9.3 (+)
- net P7: now also RV10.2, U8.12 (+); no longer RV8.2, U9.5 (+)
- net P8: now also RV13.2, U10.3 (+); no longer RV9.2, U8.10 (+)
- net P9: now also RV14.2, U10.5 (+); no longer RV10.2, U8.12 (+)
- net USB_VBUS: now also R6.2
- net at Q1.3 (C), R57.1: now also R66.1
- net at F1.2: now also S1.2 (COM_1)
- new net: D3.2 (A), R6.1
- new net: J14.5, R66.2
- new net: J14.4, R63.1
- new net +5V: R4.2, R58.1, R63.2
- no-connect marks 34 -> 45
Other:
- moved on the sheet: C10, U2
