File: Hardware/Kicad/rev0.2/Faderbay.kicad_pcb (KiCad board)
At the start: 4 copper layers, 360 x 140 mm, 182 parts, among them J1 UART, J2 USB_C_Receptacle_USB2.0_14P, J3 SWD, Q1 MMBT2222A, SW1 SW_Push_Dual, SW2 SW_Push_Dual, SW3 EC11E15204A3, SW4 SW_Push_Dual, SW5 SW_Push_Dual, SW6 SW_SPST, U1 USBLC6-2SC6, U10 MCP6004, U11 74AHCT125, U2 MCP6001-OT, U3 TLV75733PDBV, U4 STM32F405RGTx, U5 CD74HC4067M, U6 ICL7660, U7 MCP6004, U8 MCP6004, U9 MCP6004, Y1 16MHz

Commit message: Add WQP729JH jack footprints, 3D models and update rev0.2 design
Parts:
- removed C27: 100n, Capacitor_SMD:C_0402_1005Metric
- removed DS1: NHD-14432WG-BTFH-V_T, footprints:LCD_NHD-14432WG-BTFH-V_T
- removed U11: 74AHCT125, Package_SO:SOIC-14_3.9x8.7mm_P1.27mm
- added C28: 4.7u, Capacitor_SMD:C_0805_2012Metric, F.Cu at (-159.5, -44.0)
- added C29: 22p, Capacitor_SMD:C_0402_1005Metric, F.Cu at (-167.5, -43.5)
- added C39: 4.7u, Capacitor_SMD:C_0805_2012Metric, F.Cu at (-167.5, -45.5)
- added C40: 1u, Capacitor_SMD:C_0603_1608Metric, F.Cu at (-144.0, -57.1)
- added C41: 10u, Capacitor_SMD:C_0603_1608Metric, F.Cu at (-135.8, -57.0)
- added C42: 10u, Capacitor_SMD:C_0603_1608Metric, F.Cu at (-134.1, -57.0)
- added D3: MBR0520L, Diode_SMD:D_0805_2012Metric, F.Cu at (-167.9, -48.9)
- added J4: Conn_01x24, Connector_FFC-FPC:Jushuo_AFC07-S24FCA-00_1x24-1MP_P0.50_Horizontal, F.Cu at (-140.2, -51.9)
- added L1: 10u, Inductor_SMD:L_Sunlord_SWPA4030S, F.Cu at (-163.5, -50.5)
- added R6: 470, Resistor_SMD:R_0603_1608Metric, F.Cu at (123.5, -52.5)
- added R63: 1M, Resistor_SMD:R_0402_1005Metric, F.Cu at (-167.5, -42.0)
- added R65: 115k, Resistor_SMD:R_0402_1005Metric, F.Cu at (-164.7, -42.4)
- added R66: 100k, Resistor_SMD:R_0603_1608Metric, F.Cu at (-161.5, -42.0)
- added R72: 750k, Resistor_SMD:R_0603_1608Metric, F.Cu at (-137.6, -57.0)
- added U12: TPS61040DBV, Package_TO_SOT_SMD:SOT-23-5, F.Cu at (-163.5, -46.0)
- J10, J11, J12, J13, J15, J16, J17, J18, J19, J20, J21, J22, J5, J6, J7, J8: footprint footprints:PJ-320B -> footprints:WQP729JH-R
- J9: footprint footprints:PJ-320B -> footprints:WQP729JH-B
- R5: value 150 -> 1k
- U5: value CD74HC4067M -> CD74HCT4067M
- moved R65 26.2 mm to (-159.0, -47.0)
- moved R57 8.36 mm to (107.5, -56.1)
- moved R41 7.79 mm to (8.00, -53.5), turned to 0 degrees
- moved R40 6.86 mm to (5.50, -57.5), turned to 0 degrees
- moved R42 6.45 mm to (25.5, -54.0), turned to 0 degrees
- moved J17 6.07 mm to (40.5, -74.4)
- moved J10 6.07 mm to (-34.5, -74.5)
- moved J11 6.07 mm to (-22.0, -74.5)
- moved J12 6.07 mm to (-9.50, -74.5)
- moved J13 6.07 mm to (3.00, -74.5)
- moved J15 6.07 mm to (15.5, -74.5)
- moved J16 6.07 mm to (28.0, -74.5)
- moved J18 6.07 mm to (53.0, -74.5)
- moved J19 6.07 mm to (65.5, -74.5)
- moved J20 6.07 mm to (78.0, -74.5)
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Connections:
- C24 pad 1: Net-(C24-Pad1) -> VDDA
- C25 pad 1: Net-(C24-Pad1) -> GNDA
- FB3 pad 2: Net-(C24-Pad1) -> VDDA
- U4 pad 21: SPI_SCK -> DISP_SCLK
- U4 pad 26: unconnected-(U4-PB0-Pad26) -> DISP_EN
- U4 pad 27: unconnected-(U4-PB1-Pad27) -> DISP_RES
- U4 pad 29: unconnected-(U4-PB10-Pad29) -> DISP_DC
- U4 pad 42: USB_VBUS -> unconnected-(U4-PA9-Pad42)
- U4 pad 57: SPI_MOSI -> DISP_MOSI
- U6 pad 7: +5VA -> unconnected-(U6-OSC-Pad7)
Routing:
- net +5VD: track 539.5 -> 0.00 mm, vias 7 -> 0
- net SPI_MOSI: track 257.6 -> 0.00 mm, vias 2 -> 0
- net SPI_SCK: track 249.8 -> 0.00 mm, vias 2 -> 0
- net DISP_CS: track 242.7 -> 49.8 mm
- net DISP_SCLK: track 0.00 -> 80.8 mm, vias 0 -> 2
- net DISP_MOSI: track 0.00 -> 70.8 mm, vias 0 -> 2
- net SCLK: track 65.8 -> 0.00 mm, vias 1 -> 0
- net SID: track 62.5 -> 0.00 mm, vias 3 -> 0
- net ~CS: track 61.0 -> 0.00 mm, vias 3 -> 0
- net GNDA: track 822.7 -> 872.2 mm, vias 29 -> 27
- net Net-(R16-Pad2): track 44.6 -> 16.8 mm
- net Net-(DS1-LED+): track 17.8 -> 0.00 mm
- net Net-(R19-Pad2): track 51.4 -> 37.6 mm
- net Net-(Q1-C): track 5.66 -> 0.00 mm
- net Net-(J9-Pad3): track 5.56 -> 11.2 mm
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- added copper zone on F.Cu, net +12V
- added copper zone on F.Cu, net +5VD
- added copper zone on F.Cu, net Net-(D3-A)
- added copper zone on F.Cu, net Net-(U12-FB)
