File: Hardware/Kicad/rev0.2/Faderbay.kicad_sch (KiCad schematic)
At the start: 178 parts, among them J1 UART, J2 USB_C_Receptacle_USB2.0_14P, J3 SWD, Q1 MMBT2222A, SW1 SW_Push_Dual, SW2 SW_Push_Dual, SW3 EC11E15204A3, SW4 SW_Push_Dual, SW5 SW_Push_Dual, SW6 SW_SPST, U1 USBLC6-2SC6, U10 MCP6004, U11 74AHCT125, U2 MCP6001-OT, U3 TLV75733PDBV, U4 STM32F405RGTx, U5 CD74HC4067M, U6 ICL7660, U7 MCP6004, U8 MCP6004, U9 MCP6004, Y1 16MHz

Commit message: Update schematic
Parts:
- added R6: 470, symbol Device:R_Small
- R5: value 150 -> 1k
- U5: value CD74HC4067M -> CD74HCT4067M
Connections:
- net +5VA: no longer U6.7 (OSC)
- net +5VD: now also R6.1
- net GNDA: now also C25.1
- net VDDA: now also C24.1, FB3.2
- net at Q1.3 (C), R57.1: now also R6.2
- net USB_VBUS: no longer names the net of U4.42 (PA9)
- no-connect marks 34 -> 36
Other:
- note added: "Pendiente de testear ripple"
- moved on the sheet: C24, C25, C26, J9, Q1, R57, R58, R64, TP7

Commit message: Add WQP729JH jack footprints, 3D models and update rev0.2 design
Parts:
- removed C27: 100n, Capacitor_SMD:C_0402_1005Metric, symbol Device:C_Small
- removed DS1: NHD-14432WG-BTFH-V_T, footprints:LCD_NHD-14432WG-BTFH-V_T, symbol User:NHD-14432WG-BTFH-V_T
- removed U11: 74AHCT125, Package_SO:SOIC-14_3.9x8.7mm_P1.27mm, symbol 74xx:74AHCT125
- added C28, C39: 4.7u, Capacitor_SMD:C_0805_2012Metric, symbol Device:C_Small
- added C29: 22p, Capacitor_SMD:C_0402_1005Metric, symbol Device:C_Small
- added C40: 1u, Capacitor_SMD:C_0603_1608Metric, symbol Device:C_Small
- added C41, C42: 10u, Capacitor_SMD:C_0603_1608Metric, symbol Device:C_Small
- added D3: MBR0520L, Diode_SMD:D_0805_2012Metric, symbol Device:D_Schottky_Small
- added J4: Conn_01x24, Connector_FFC-FPC:Jushuo_AFC07-S24FCA-00_1x24-1MP_P0.50_Horizontal, symbol Connector_Generic:Conn_01x24
- added L1: 10u, Inductor_SMD:L_Sunlord_SWPA4030S, symbol Device:L_Small
- added R63: 1M, Resistor_SMD:R_0402_1005Metric, symbol Device:R_Small
- added R66: 100k, Resistor_SMD:R_0603_1608Metric, symbol Device:R_Small
- added R72: 750k, Resistor_SMD:R_0603_1608Metric, symbol Device:R_Small
- added U12: TPS61040DBV, Package_TO_SOT_SMD:SOT-23-5, symbol Regulator_Switching:TPS61040DBV
- J10, J11, J12, J13, J15, J16, J17, J18, J19, J20, J21, J22, J5, J6, J7, J8: footprint footprints:PJ-320B -> footprints:WQP729JH-R; symbol Eurorack:PJ-320B -> Eurorack:WQP729JH-R; MP PJ-320B -> WQP729JH-R
- J9: footprint footprints:PJ-320B -> footprints:WQP729JH-B; symbol Eurorack:PJ-320B -> Eurorack:WQP729JH-B; MP PJ-320B -> WQP729JH-B
- R6: footprint (none) -> Resistor_SMD:R_0603_1608Metric
- R65: value 56 -> 115k; footprint Resistor_SMD:R_0805_2012Metric -> Resistor_SMD:R_0402_1005Metric
Connections:
- net +3.3V: now also C40.1, J4.5 (Pin_5)
- net +5VD: now also C28.1, L1.1, U12.5 (VIN); no longer R65.1
- net DISP_CS: now also J4.8 (Pin_8)
- net GNDA: now also J10.4, J11.4, J12.4, J13.4, J15.4, J16.4, J17.4, J18.4, J19.4, J20.4, J21.4, J22.4, J5.4, J6.4, J7.4, J8.4; no longer J10.2, J11.2, J12.2, J13.2, J15.2, J16.2, J17.2, J18.2, J19.2, J20.2, J21.2, J22.2, J5.2, J6.2, J7.2, J8.2
- net GNDD: now also R65.2, C28.2, C39.2, C40.2, C41.2, C42.2, J4.1 (Pin_1), J4.11 (Pin_11), J4.12 (Pin_12), J4.16 (Pin_16), J4.17 (Pin_17), J4.18 (Pin_18), J4.19 (Pin_19), J4.2 (Pin_2), J4.20 (Pin_20), J4.24 (Pin_24), J4.3 (Pin_3), J4.6 (Pin_6), J4.7 (Pin_7), R66.2, R72.1, U12.2 (GND)
- net at J9.3, R57.2: now also J9.4
- net DISP_EN: now reaches U4.26 (PB0)
- net DISP_EN: now also R66.1, U12.4 (EN)
- net DISP_RES: now reaches U4.27 (PB1)
- net DISP_RES: now also J4.9 (Pin_9)
- net DISP_DC: now reaches U4.29 (PB10)
- net DISP_DC: now also J4.10 (Pin_10)
- net SPI_MOSI renamed DISP_MOSI
- net DISP_MOSI: now also J4.14 (Pin_14)
- net SPI_SCK renamed DISP_SCLK
- net DISP_SCLK: now also J4.13 (Pin_13)
- new net: D3.2 (A), L1.2, U12.1 (SW)
- new net: C29.2, R63.2, R65.1, U12.3 (FB)
- new net: C41.1, J4.22 (Pin_22)
- new net: J4.21 (Pin_21), R72.2
- new net +12V: C29.1, C39.1, C42.1, D3.1 (K), J4.23 (Pin_23), R63.1
- no-connect marks 36 -> 32
Other:
- note added: "12V BOOST"
- moved on the sheet: C20, C21, C24, C25, C26, C30, C31, C32, C33, C34, C35, C36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
